File: hardware/Eagle files/untitled.sch (EAGLE design)
At the start: 35 parts

Commit message: Updated to revision 2
All files updated to revision 2 of the ECMeter. New code and hardware
files added.
Parts:
- removed C15: 1uF, SparkFun-Capacitors:CAP0805
- removed MCP9700AT: MCP9700AT, benkyo:MCP9700AT-E/LT
- removed U$4: MCP3426, benkyo:MCP3426
- added C17, C19: 2.2nF, SparkFun-Capacitors:CAP0603-CAP
- added C18, C20: 4.7uF, SparkFun-Capacitors:CAP0805
- added MCP3428: MCP3428, benkyo:MCP3428
- added R11: 3K, SparkFun-Resistors:1K-1%
- added R12: 20.5K, SparkFun-Resistors:1K-1%
- added R13: 10K, SparkFun-Resistors:1K-1%
- added SJ1: SOLDERJUMPERNO, SparkFun-Retired:SOLDERJUMPERNO
- added U$5: MCP9700AT-E/TT, benkyo:MCP9700AT-E/TT
- C1: value 10uF -> 22uF
- C10, C12, C13, C14, C16, C2: value 1uF -> 0.1uF; device SparkFun-Capacitors:CAP0805 -> SparkFun-Capacitors:CAP0603-CAP
- C11, C3, C4, C7, C8, C9: device SparkFun-Capacitors:CAP0805 -> SparkFun-Capacitors:CAP0603-CAP
- C5, C6: value 10nF -> 0.1uF
- D2: value (none) -> Schottky
- JP1: device SparkFun-Connectors:M04POLAR -> SparkFun-Connectors:M04LONGPADS
- R1: value 1k -> 51K
- R2, R6, R7: value 1k -> 1K
- R4: value 100k -> 51K
- R5: value 10k -> 10K
- R9: value 100k -> 1M
- U$1: value TL072A -> TLC272CD
- U$2: device benkyo:K1-PROBE -> benkyo2:K1-PROBE
Connections:
- removed net ADC_EC_IN: C10.1, C11.1, D2.C, R9.2, U$1G$2.-IN, U$4.CH1+
- removed net N$46: C9.2, MCP9700AT.VOUT, U$4.CH2+
- new net ADC_EC: C16.1, C7.1, D2.C, MCP3428.CH1+, R9.2, U$1G$2.-IN
- new net ADC_TEMP: C11.1, MCP3428.CH3+, U$5.VOUT
- new net ADC_VOLTAGE: MCP3428.CH4+, R12.2, R13.1
- new net N$48: C19.2, R1.2, R4.1
- new net N$50: MCP3428.ADR1, SJ1.1
- net GND: now also C10.1, C12.1, C13.1, C14.1, C17.1, C18.1, C19.1, C2.1, C20.2, C3.2, C4.1, JP1.1, MCP3428.CH1-, MCP3428.CH2-, MCP3428.CH3-, MCP3428.CH4-, MCP3428.GND, R11.2, R13.2, SJ1.2, U$5.GND; no longer C10.2, C12.2, C13.2, C14.2, C15.2, C2.2, C3.1, C4.2, JP1.4, MCP9700AT.GND, R1.1, U$4.CH1-, U$4.CH2-, U$4.GND
- net N$13: now also C8.1; no longer C8.2
- net N$14: now also C8.2; no longer C8.1
- net N$6: now also C17.2, R1.1, R11.1; no longer R1.2, R4.1
- net SCL: now also JP1.4, MCP3428.SCL; no longer JP1.1, U$4.SCL
- net SDA: now also JP1.3, MCP3428.SDA; no longer JP1.2, U$4.SDA
- net VCC: now also C10.2, C12.2, C2.2, C20.1, C4.2, C9.2, JP1.2, MCP3428.ADR0, MCP3428.VCC, R12.1, U$5.VDD; no longer C12.1, C13.1, C16.1, C2.1, C4.1, C7.1, JP1.3, MCP9700AT.VDD, U$4.VCC
- net VNEG: now also C13.2, C14.2, C18.2, C3.1; no longer C14.1, C15.1, C3.2
Other:
- note added: "Pull-up resistors not needed when master has them"
- note added: "Voltage divider and second order low-pass filter"
- note added: "Voltage measurement"
- note added: "Wien bridge oscillator @ ~1.6Khz"
- note removed: "Wien bridge oscillator @ ~16Khz"
- moved on the sheet: C1, C10, C11, C12, C13, C14, C16, C2, C3, C4, C7, C8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
